File: RM2025_G473_MCB_StdExtend/RM2025_G473_MCB_StdExtend.kicad_pcb (KiCad board)
At the start: 2 copper layers, 60 x 40 mm, 54 parts, among them J1 RS-485, J10 GPIO1, J11 GPIO1, J12 BTB, J13 CAN, J14 RS-485, J15 CAN, J16 CAN, J17 CAN, J18 Conn_01x07_MountingPin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

Commit message: ibom和加工文件
Parts:
- J10, J11, J2, J3: value GPIO1 -> GPIO
Other:
- board text added: "洗板别太久"
- board text removed: "个是横的"
- board text removed: "了"
- board text removed: "些"
- board text removed: "侯"
- board text removed: "口"
- board text removed: "接"
- board text removed: "时"
- board text removed: "洗版别太久"
- board text removed: "焊"
- board text removed: "焊的时候看好了这个是有方向的 LED也有方向"
- board text removed: "的"
- board text removed: "看好"
- board text removed: "竖"
- board text removed: "竖的"
- board text removed: "这"
- board text removed: "这两"
- board text removed: "都是"
