File: RM2025_G473_MCB_StdExtend/RM2025_G473_MCB_StdExtend.kicad_sch (KiCad schematic)
At the start: 53 parts, among them J1 RS-485, J10 GPIO1, J11 GPIO1, J12 BTB, J13 CAN, J14 RS-485, J15 CAN, J16 CAN, J17 CAN, J18 Conn_01x07_MountingPin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

Commit message: ibom和加工文件
Parts:
- J10, J11, J2, J3: value GPIO1 -> GPIO
Other:
- note removed: "FLASH"
- note removed: "Layout & Connectors"
- note removed: "Partly modified from F Board by Jason Chan and JYC"
- note removed: "Peripherals"
- note removed: "Please refer to "RM G473 CShape Manuel" for more information"
- note removed: "RM G473 CShape V24.02"
- note removed: "SWD"
- note removed: "zxianaa@connect.ust.hk"
- moved on the sheet: C1, C2, C3, C4, C5, C6, C7, C78, D1, D2, D3, D4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
